Commit message: urdf的j2和j3抬起2度

File: src/piper_description/urdf/piper_description_old.urdf (robot description, URDF)
Before this commit: robot piper, 10 links, 9 joints
Joints:
- joint joint2: origin xyz=0 0 0 rpy=1.5708 -0.1259 -3.1416 -> xyz=0 0 0 rpy=1.5708 -0.10095 -3.1416
- joint joint3: origin xyz=0.28503 0 0 rpy=0 0 -1.7939 -> xyz=0.28503 0 0 rpy=0 0 -1.759

File: src/piper_description/urdf/piper_no_gripper_description.urdf (robot description, URDF)
Before this commit: robot piper, 7 links, 6 joints
Joints:
- joint joint2: origin xyz=0 0 0 rpy=1.5708 -0.10095 -3.1416 -> xyz=0 0 0 rpy=1.5708 -0.1359 -3.1416
- joint joint3: origin xyz=0.28503 0 0 rpy=0 0 -1.759 -> xyz=0.28503 0 0 rpy=0 0 -1.7939

File: src/piper_description/urdf/piper_no_gripper_description_old.urdf (robot description, URDF)
Before this commit: robot piper, 10 links, 9 joints
Links:
- removed link gripper_base
- removed link link7
- removed link link8
Joints:
- removed joint joint6_to_gripper_base
- removed joint joint7
- removed joint joint8
- joint joint2: origin xyz=0 0 0 rpy=1.5708 -0.1259 -3.1416 -> xyz=0 0 0 rpy=1.5708 -0.10095 -3.1416
- joint joint3: origin xyz=0.28503 0 0 rpy=0 0 -1.7939 -> xyz=0.28503 0 0 rpy=0 0 -1.759
- joint joint6: limit lower=-2.0944 upper=2.0944 effort=100 velocity=3 -> lower=-2.0944 upper=2.0944 effort=100 velocity=5
