Commit message: [BUG]勘误urdf中joint1关节的正方向角度限制为2.168rad的错误,应为2.618rad(150度)

File: src/piper_description/urdf/piper_description.xacro (robot description, xacro)
@@ -104,5 +104,5 @@
     <limit
       lower="-2.618"
-      upper="2.168"
+      upper="2.618"
       effort="100"
       velocity="5" />

File: src/piper_description/urdf/piper_description_old.urdf (robot description, URDF)
Before this commit: robot piper, 10 links, 9 joints
Joints:
- joint joint1: limit lower=-2.618 upper=2.168 effort=100 velocity=5 -> lower=-2.618 upper=2.618 effort=100 velocity=5

File: src/piper_description/urdf/piper_no_gripper_description.urdf (robot description, URDF)
Before this commit: robot piper, 8 links, 7 joints
Joints:
- joint joint1: limit lower=-2.618 upper=2.168 effort=100 velocity=5 -> lower=-2.618 upper=2.618 effort=100 velocity=5

File: src/piper_description/urdf/piper_no_gripper_description.xacro (robot description, xacro)
@@ -104,5 +104,5 @@
     <limit
       lower="-2.618"
-      upper="2.168"
+      upper="2.618"
       effort="100"
       velocity="5" />

File: src/piper_description/urdf/piper_no_gripper_description_old.urdf (robot description, URDF)
Before this commit: robot piper, 7 links, 6 joints
Joints:
- joint joint1: limit lower=-2.618 upper=2.168 effort=100 velocity=5 -> lower=-2.618 upper=2.618 effort=100 velocity=5
