Commit message: ✨ feat(piper_description_with_teach): 修改示教器的质量重心和惯性张量参数，修改gripper_base为teach_base

File: src/piper_description/urdf/piper_description_with_teach.urdf (robot description, URDF)
Before this commit: robot piper, 10 links, 9 joints
Links:
- removed link gripper_base
- added link teach_base, mass 0.5; collision mesh filename=package://piper_description/meshes/teach_base.STL; visual mesh filename=package://piper_description/meshes/teach_base.STL
- link link7: mass 0.025 -> 0.02
- link link8: mass 0.025 -> 0.02
Joints:
- removed joint joint6_to_gripper_base
- added joint joint6_to_teach_base: type fixed, parent link6, child teach_base, origin xyz=0 0 0 rpy=0 0 0
- joint joint7: parent gripper_base -> teach_base
- joint joint8: parent gripper_base -> teach_base
