Commit message: [FIXED]修改urdf为最新版本,对应固件1.6-3以上

File: src/piper_description/urdf/piper_description.urdf (robot description, URDF)
Before this commit: robot piper, 10 links, 9 joints
Joints:
- joint joint2: origin xyz=0 0 0 rpy=1.5708 -0.1259 -3.1416 -> xyz=0 0 0 rpy=1.5708 -0.1359 -3.1416

File: src/piper_description/urdf/piper_description.xacro (robot description, xacro)
@@ -126,5 +126,6 @@
     <origin
       xyz="0 0 0"
-      rpy="1.5708 -0.10095 -3.1416" />
+      rpy="1.5708 -0.1359 -3.1416" />
+      <!-- rpy="1.5708 -0.10095-0.03490659 -3.1416" /> -->
     <parent
       link="link1" />
@@ -175,5 +176,6 @@
     <origin
       xyz="0.28503 0 0"
-      rpy="0 0 -1.759" />
+      rpy="0 0 -1.7939" />
+      <!-- rpy="0 0 -1.759-0.03490659" /> -->
     <parent
       link="link2" />

File: src/piper_description/urdf/piper_description_gazebo.xacro (robot description, xacro)
@@ -126,5 +126,6 @@
     <origin
       xyz="0 0 0"
-      rpy="1.5708 -0.10095 -3.1416" />
+      rpy="1.5708 -0.1359 -3.1416" />
+      <!-- rpy="1.5708 -0.10095-0.03490659 -3.1416" /> -->
     <parent
       link="link1" />
@@ -175,5 +176,6 @@
     <origin
       xyz="0.28503 0 0"
-      rpy="0 0 -1.759" />
+      rpy="0 0 -1.7939" />
+      <!-- rpy="0 0 -1.759-0.03490659" /> -->
     <parent
       link="link2" />

File: src/piper_description/urdf/piper_no_gripper_description.xacro (robot description, xacro)
@@ -126,5 +126,6 @@
     <origin
       xyz="0 0 0"
-      rpy="1.5708 -0.10095 -3.1416" />
+      rpy="1.5708 -0.1359 -3.1416" />
+      <!-- rpy="1.5708 -0.10095-0.03490659 -3.1416" /> -->
     <parent
       link="link1" />
@@ -175,5 +176,6 @@
     <origin
       xyz="0.28503 0 0"
-      rpy="0 0 -1.759" />
+      rpy="0 0 -1.7939" />
+      <!-- rpy="0 0 -1.759-0.03490659" /> -->
     <parent
       link="link2" />

File: src/piper_description/urdf/piper_no_gripper_description_gazebo.xacro (robot description, xacro)
@@ -126,5 +126,6 @@
     <origin
       xyz="0 0 0"
-      rpy="1.5708 -0.10095 -3.1416" />
+      rpy="1.5708 -0.1359 -3.1416" />
+      <!-- rpy="1.5708 -0.10095-0.03490659 -3.1416" /> -->
     <parent
       link="link1" />
@@ -175,5 +176,6 @@
     <origin
       xyz="0.28503 0 0"
-      rpy="0 0 -1.759" />
+      rpy="0 0 -1.7939" />
+      <!-- rpy="0 0 -1.759-0.03490659" /> -->
     <parent
       link="link2" />

Commit message: 🎈 perf(urdf): 修改夹爪力矩最大值为100

File: src/piper_description/urdf/piper_description.urdf (robot description, URDF)
Before this commit: robot piper, 11 links, 10 joints
Joints:
- joint joint7: limit lower=0 upper=0.035 effort=10 velocity=1 -> lower=0 upper=0.035 effort=100 velocity=1
- joint joint8: limit lower=-0.035 upper=0 effort=10 velocity=1 -> lower=-0.035 upper=0 effort=100 velocity=1

File: src/piper_description/urdf/piper_description.xacro (robot description, xacro)
@@ -506,5 +506,5 @@
       lower="0"
       upper="0.035"
-      effort="10"
+      effort="100"
       velocity="1" />
   </joint>
@@ -564,5 +564,5 @@
       lower="-0.035"
       upper="0"
-      effort="10"
+      effort="100"
       velocity="1" />
   </joint>

File: src/piper_description/urdf/piper_description_old.urdf (robot description, URDF)
Before this commit: robot piper, 10 links, 9 joints
Joints:
- joint joint7: limit lower=0 upper=0.035 effort=10 velocity=1 -> lower=0 upper=0.035 effort=100 velocity=1
- joint joint8: limit lower=-0.035 upper=0 effort=10 velocity=1 -> lower=-0.035 upper=0 effort=100 velocity=1

Commit message: 🐞 fix(urdf、meshes): 更新urdf文件

File: src/piper_description/urdf/piper_description.urdf (robot description, URDF)
Before this commit: robot piper_description, 9 links, 8 joints
Links:
- added link gripper_base, mass 0.45; collision mesh filename=package://piper_description/meshes/gripper_base.STL; visual mesh filename=package://piper_description/meshes/gripper_base.STL
- link base_link: mass None -> 1.02
- link link1: mass 0.0978679932242825 -> 0.71
- link link2: mass 0.289571136953082 -> 1.17
- link link3: mass 0.290583247455324 -> 0.5
- link link4: mass 0.127087348341362 -> 0.38
- link link5: mass 0.144711209371719 -> 0.383
- link link6: mass 0.150196458571266 -> 0.00699089613564366
- link link7: mass 0.0264822500394006 -> 0.025
- link link8: mass 0.0264822490707451 -> 0.025
Joints:
- added joint joint6_to_gripper_base: type fixed, parent link6, child gripper_base, origin xyz=0 0 0 rpy=0 0 0
- joint joint1: limit lower=-2.618 upper=2.618 effort=100 velocity=0 -> lower=-2.618 upper=2.168 effort=100 velocity=5; origin xyz=0 0 0.123 rpy=0 0 -1.5708 -> xyz=0 0 0.123 rpy=0 0 0
- joint joint2: limit lower=0 upper=3.14 effort=100 velocity=1 -> lower=0 upper=3.14 effort=100 velocity=5; origin xyz=0 0 0 rpy=1.5708 -0.10095 -1.5708 -> xyz=0 0 0 rpy=1.5708 -0.1359 -3.1416
- joint joint3: limit lower=-2.967 upper=0 effort=100 velocity=1 -> lower=-2.967 upper=0 effort=100 velocity=5; origin xyz=0.28503 0 0 rpy=0 0 1.3826 -> xyz=0.28503 0 0 rpy=0 0 -1.7939
- joint joint4: axis 0 0 -1 -> 0 0 1; limit lower=-1.832 upper=1.832 effort=100 velocity=1 -> lower=-1.745 upper=1.745 effort=100 velocity=5; origin xyz=0.021984 0.25075 0 rpy=-1.5708 0 0 -> xyz=-0.021984 -0.25075 0 rpy=1.5708 0 0
- joint joint5: limit lower=-1.22 upper=1.22 effort=100 velocity=1 -> lower=-1.22 upper=1.22 effort=100 velocity=5; origin xyz=0 0 0 rpy=1.5708 -0.087266 0 -> xyz=0 0 0 rpy=-1.5708 0 0
- joint joint6: axis 0 0 -1 -> 0 0 1; limit lower=-3.14 upper=3.14 effort=100 velocity=1 -> lower=-2.0944 upper=2.0944 effort=100 velocity=3; origin xyz=0 0.091 0.0014165 rpy=-1.5708 -1.5708 0 -> xyz=8.8259E-05 -0.091 0 rpy=1.5708 0 0
- joint joint7: axis 0 0 -1 -> 0 0 1; limit lower=-0.038 upper=0 effort=100 velocity=1 -> lower=0 upper=0.035 effort=10 velocity=1; origin xyz=0 0 0.13503 rpy=1.5708 0 1.5708 -> xyz=0 0 0.1358 rpy=1.5708 0 0; parent link6 -> gripper_base
- joint joint8: axis 0 0 1 -> 0 0 -1; limit lower=0 upper=0.038 effort=100 velocity=1 -> lower=-0.035 upper=0 effort=10 velocity=1; origin xyz=0 0 0.13503 rpy=-1.5708 0 1.5708 -> xyz=0 0 0.1358 rpy=1.5708 0 -3.1416; parent link6 -> gripper_base

File: src/piper_description/urdf/piper_description.xacro (robot description, xacro)
@@ -10,19 +10,10 @@
   </joint>
 <!-- arm -->
-  <link
+<link
     name="base_link">
     <inertial>
-      <origin
-        xyz="-0.00973928490005031 1.8312708928633E-06 0.0410140167677137"
-        rpy="0 0 0" />
-      <mass
-        value="0.00001" />
-      <inertia
-        ixx="0.000226592553127906"
-        ixy="-7.33974356968813E-08"
-        ixz="2.13221970218123E-06"
-        iyy="0.000269447877479622"
-        iyz="8.15167478685076E-09"
-        izz="0.000222318286704" />
+            <origin xyz="-0.00473641164191482 2.56829134630247E-05 0.041451518036016" rpy="0 0 0" />
+            <mass value="1.02" />
+            <inertia ixx="0.00267433" ixy="-0.00000073" ixz="-0.00017389" iyy="0.00282612" iyz="0.0000004" izz="0.00089624" />
     </inertial>
     <visual>
@@ -53,16 +44,7 @@
     name="link1">
     <inertial>
-      <origin
-        xyz="0.00131676031927021 0.000310288842008364 -0.00922874512303438"
-        rpy="0 0 0" />
-      <mass
-        value="0.00001" />
-      <inertia
-        ixx="7.76684558296781E-05"
-        ixy="1.09084650459916E-07"
-        ixz="-1.97480532432411E-06"
-        iyy="9.24967780161546E-05"
-        iyz="9.91284646834672E-07"
-        izz="8.24589062407806E-05" />
+            <origin xyz="0.000121504734057468 0.000104632162460536 -0.00438597309559853" rpy="0 0 0" />
+            <mass value="0.71" />
+            <inertia ixx="0.00048916" ixy="-0.00000036" ixz="-0.00000224" iyy="0.00040472" iyz="-0.00000242" izz="0.00043982" />
     </inertial>
     <visual>
@@ -95,5 +77,5 @@
     <origin
       xyz="0 0 0.123"
-      rpy="0 0 -1.5708" />
+      rpy="0 0 0" />
     <parent
       link="base_link" />
@@ -104,23 +86,14 @@
     <limit
       lower="-2.618"
-      upper="2.618"
+      upper="2.168"
       effort="100"
-      velocity="1" />
+      velocity="5" />
   </joint>
   <link
     name="link2">
     <inertial>
-      <origin
-        xyz="0.147615838821413 -0.0174259998251393 0.00175952516190707"
-        rpy="0 0 0" />
-      <mass
-        value="0.00001" />
-      <inertia
-        ixx="0.000150112628108228"
-        ixy="8.58974959950769E-05"
-        ixz="-1.07428153464285E-06"
-        iyy="0.00172585302855383"
-        iyz="-9.93704792239686E-07"
-        izz="0.00177445942914759" />
+            <origin xyz="0.198666145229743 -0.010926924140076 0.00142121714502687" rpy="0 0 0" />
+            <mass value="1.17" />
+            <inertia ixx="0.00116918" ixy="-0.00180037" ixz="0.00025146" iyy="0.06785384" iyz="-0.00000455" izz="0.06774489" />
     </inertial>
     <visual>
@@ -153,5 +126,6 @@
     <origin
       xyz="0 0 0"
-      rpy="1.5708 -0.10095 -1.5708" />
+      rpy="1.5708 -0.1359 -3.1416" />
+      <!-- rpy="1.5708 -0.10095-0.03490659 -3.1416" /> -->
     <parent
       link="link1" />
@@ -164,21 +138,12 @@
       upper="3.14"
       effort="100"
-      velocity="1" />
+      velocity="5" />
   </joint>
   <link
     name="link3">
     <inertial>
-      <origin
-        xyz="0.0156727246030052 0.104466514905741 0.000508486764144372"
-        rpy="0 0 0" />
-      <mass
-        value="0.00001" />
-      <inertia
-        ixx="0.000221686352136266"
-        ixy="-7.57426543992343E-06"
-        ixz="-6.3700062772173E-07"
-        iyy="0.000100859162015934"
-        iyz="-8.16202696860781E-07"
-        izz="0.000241839316548946" />
+            <origin xyz="-0.0202737662122021 -0.133914995944595 -0.000458682652737356" rpy="0 0 0" />
+            <mass value="0.5" />
+            <inertia ixx="0.01361711" ixy="0.00165794" ixz="-0.00000048" iyy="0.00045024" iyz="-0.00000045" izz="0.01380322" />
     </inertial>
     <visual>
@@ -211,5 +176,6 @@
     <origin
       xyz="0.28503 0 0"
-      rpy="0 0 1.3826" />
+      rpy="0 0 -1.7939" />
+      <!-- rpy="0 0 -1.759-0.03490659" /> -->
     <parent
       link="link2" />
@@ -222,21 +188,12 @@
       upper="0"
       effort="100"
-      velocity="1" />
+      velocity="5" />
   </joint>
   <link
     name="link4">
     <inertial>
-      <origin
-        xyz="0.000276464622388145 -0.00102803669324853 -0.00472830700561612"
-        rpy="0 0 0" />
-      <mass
-        value="0.00001" />
-      <inertia
-        ixx="3.82011730423098E-05"
-        ixy="-4.92358351033589E-08"
-        ixz="4.89589432983109E-08"
-        iyy="4.87048555222491E-05"
-        iyz="6.70802942486707E-08"
-        izz="4.10592077565155E-05" />
+            <origin xyz="-9.66635791618542E-05 0.000876064475651083 -0.00496880904640868" rpy="0 0 0" />
+            <mass value="0.38" />
+            <inertia ixx="0.00018501" ixy="0.00000054" ixz="0.00000120" iyy="0.00018965" iyz="-0.00000841" izz="0.00015484" />
     </inertial>
     <visual>
@@ -268,6 +225,6 @@
     type="revolute">
     <origin
-      xyz="0.021984 0.25075 0"
-      rpy="-1.5708 0 0" />
+      xyz="-0.021984 -0.25075 0"
+      rpy="1.5708 0 0" />
     <parent
       link="link3" />
@@ -275,26 +232,17 @@
       link="link4" />
     <axis
-      xyz="0 0 -1" />
-    <limit
-      lower="-1.832"
-      upper="1.832"
+      xyz="0 0 1" />
+    <limit
+      lower="-1.745"
+      upper="1.745"
       effort="100"
-      velocity="1" />
+      velocity="5" />
   </joint>
   <link
     name="link5">
     <inertial>
-      <origin
-        xyz="8.82261259100015E-05 0.056682908434204 -0.00196119077436732"
-        rpy="0 0 0" />
-      <mass
-        value="0.00001" />
-      <inertia
-        ixx="4.39644269159173E-05"
-        ixy="-3.59214840853815E-08"
-        ixz="-1.89785003257649E-08"
-        iyy="5.63173857792457E-05"
-        iyz="-2.15407623722543E-07"
-        izz="4.88713595021005E-05" />
+            <origin xyz="-4.10554118924211E-05 -0.0566486692356075 -0.0037205791677906" rpy="0 0 0" />
+            <mass value="0.383" />
+            <inertia ixx="0.00166169" ixy="0.00000006" ixz="-0.00000007" iyy="0.00018510" iyz="0.00001026" izz="0.00164321" />
     </inertial>
     <visual>
@@ -327,5 +275,5 @@
     <origin
       xyz="0 0 0"
-      rpy="1.5708 -0.087266 0" />
+      rpy="-1.5708 0 0" />
     <parent
       link="link4" />
@@ -338,21 +286,12 @@
       upper="1.22"
       effort="100"
-      velocity="1" />
+      velocity="5" />
   </joint>
   <link
     name="link6">
     <inertial>
-      <origin
-        xyz="9.41121070072333E-09 0.000341209775988838 0.0342122921883722"
-        rpy="0 0 0" />
-      <mass
-        value="0.00001" />
-      <inertia
-        ixx="4.31750564711759E-05"
-        ixy="-2.21295720427027E-08"
-        ixz="-3.27825836857102E-12"
-        iyy="9.99756357365307E-05"
-        iyz="1.10337380549335E-07"
-        izz="0.000118282295533688" />
+            <origin xyz="-8.82590762930069E-05 9.0598378529832E-06 -0.002" rpy="0 0 0" />
+            <mass value="0.00699089613564366" />
+            <inertia ixx="5.73015540542155E-07" ixy="-1.98305403089247E-22" ixz="-7.2791893904596E-23" iyy="5.73015540542155E-07" iyz="-3.4146026640245E-24" izz="1.06738869138926E-06" />
     </inertial>
     <visual>
@@ -367,5 +306,5 @@
         name="">
         <color
-          rgba="0.792156862745098 0.819607843137255 0.933333333333333 1" />
+          rgba="0.898039215686275 0.917647058823529 0.929411764705882 1" />
       </material>
     </visual>
@@ -384,6 +323,6 @@
     type="revolute">
     <origin
-      xyz="0 0.091 0.0014165"
-      rpy="-1.5708 -1.5708 0" />
+      xyz="8.8259E-05 -0.091 0"
+      rpy="1.5708 0 0" />
     <parent
       link="link5" />
@@ -391,10 +330,61 @@
       link="link6" />
     <axis
-      xyz="0 0 -1" />
-    <limit
-      lower="-3.14"
-      upper="3.14"
+      xyz="0 0 1" />
+    <limit
+      lower="-2.0944"
+      upper="2.0944"
       effort="100"
-      velocity="1" />
+      velocity="3" />
+  </joint>
+  <link
+    name="gripper_base">
+    <inertial>
+      <origin
+        xyz="-0.000183807162235591 8.05033155577911E-05 0.0321436689908876"
+        rpy="0 0 0" />
+      <mass
+        value="0.45" />
+      <inertia
+        ixx="0.00092934"
+        ixy="0.00000034"
+        ixz="-0.00000738"
+        iyy="0.00071447"
+        iyz="0.00000005"
+        izz="0.00039442" />
+    </inertial>
+    <visual>
+      <origin
+        xyz="0 0 0"
+        rpy="0 0 0" />
+      <geometry>
+        <mesh
+          filename="package://piper_description/meshes/gripper_base.STL" />
+      </geometry>
+      <material
+        name="">
+        <color
+          rgba="0.792156862745098 0.819607843137255 0.933333333333333 1" />
+      </material>
+    </visual>
+    <collision>
+      <origin
+        xyz="0 0 0"
+        rpy="0 0 0" />
+      <geometry>
+        <mesh
+          filename="package://piper_description/meshes/gripper_base.STL" />
+      </geometry>
+    </collision>
+  </link>
+  <joint
+    name="joint6_to_gripper_base"
+    type="fixed">
+    <origin
+      xyz="0 0 0"
+      rpy="0 0 0" />
+    <parent
+      link="link6" />
+    <child
+      link="gripper_base" />
   </joint>
   <link
@@ -402,15 +392,15 @@
     <inertial>
       <origin
-        xyz="-0.000277795893713934 -0.046767350270289 -0.00921029791141448"
+        xyz="0.00065123185041968 -0.0491929869131989 0.00972258769184025"
         rpy="0 0 0" />
       <mass
-        value="0.00001" />
+        value="0.025" />
       <inertia
-        ixx="9.99782519244544E-06"
-        ixy="-1.57547595978589E-07"
-        ixz="-2.71355785017816E-08"
-        iyy="6.17952364356547E-06"
-        iyz="-1.58939504838734E-06"
-        izz="1.42102253390315E-05" />
+        ixx="0.00007371"
+        ixy="-0.00000113"
+        ixz="0.00000021"
+        iyy="-0.00000113"
+        iyz="-0.00001372"
+        izz="0.0000747" />
     </inertial>
     <visual>
@@ -442,16 +432,16 @@
     type="prismatic">
     <origin
-      xyz="0 0 0.13503"
-      rpy="1.5708 0 1.5708" />
-    <parent
-      link="link6" />
+      xyz="0 0 0.1358"
+      rpy="1.5708 0 0" />
+    <parent
+      link="gripper_base" />
     <child
       link="link7" />
     <axis
-      xyz="0 0 -1" />
+      xyz="0 0 1" />
     <limit
       lower="0"
-      upper="0.038"
-      effort="100"
+      upper="0.035"
+      effort="10"
       velocity="1" />
   </joint>
@@ -460,15 +450,15 @@
     <inertial>
       <origin
-        xyz="0.000277795911672651 0.0467673513153836 -0.00921029799058583"
+        xyz="0.000651231850419722 -0.0491929869131991 0.00972258769184024"
         rpy="0 0 0" />
       <mass
-        value="0.00001" />
+        value="0.025" />
       <inertia
-        ixx="9.99782474142963E-06"
-        ixy="-1.57547666236405E-07"
-        ixz="2.71355834243046E-08"
-        iyy="6.17952362333486E-06"
-        iyz="1.58939503259658E-06"
-        izz="1.42102248648757E-05" />
+        ixx="0.00007371"
+        ixy="-0.00000113"
+        ixz="0.00000021"
+        iyy="-0.00000113"
+        iyz="-0.00001372"
+        izz="0.0000747" />
     </inertial>
     <visual>
@@ -500,16 +490,16 @@
     type="prismatic">
     <origin
-      xyz="0 0 0.13503"
-      rpy="-1.5708 0 1.5708" />
-    <parent
-      link="link6" />
+      xyz="0 0 0.1358"
+      rpy="1.5708 0 -3.1416" />
+    <parent
+      link="gripper_base" />
     <child
       link="link8" />
     <axis
-      xyz="0 0 1" />
-    <limit
-      lower="-0.038"
+      xyz="0 0 -1" />
+    <limit
+      lower="-0.035"
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
Commit message: 增加piper_x的模型和piper 的dea文件

File: src/piper_description/urdf/piper_description.urdf (robot description, URDF)
Before this commit: robot piper, 11 links, 10 joints
Joints:
- joint joint7: limit lower=0 upper=0.035 effort=100 velocity=1 -> lower=0 upper=0.035 effort=10 velocity=1
- joint joint8: limit lower=-0.035 upper=0 effort=100 velocity=1 -> lower=-0.035 upper=0 effort=10 velocity=1

File: src/piper_x_description/urdf/piper_x_description.urdf (robot description, URDF)
Before this commit: robot piper, 7 links, 6 joints
Links:
- link base_link: mass 1.02 -> 0.15430453053243; geometry collision mesh filename=package://piper_x_description/meshes/base_link.STL; visual mesh filename=package://piper_x_description/meshes/base_link.STL
- link link1: mass 0.71 -> 0.105313818325577; geometry collision mesh filename=package://piper_x_description/meshes/link1.STL; visual mesh filename=package://piper_x_description/meshes/link1.STL
- link link2: mass 1.17 -> 0.30648; geometry collision mesh filename=package://piper_x_description/meshes/link2.STL; visual mesh filename=package://piper_x_description/meshes/link2.STL
- link link3: mass 0.5 -> 0.16677; geometry collision mesh filename=package://piper_x_description/meshes/link3.STL; visual mesh filename=package://piper_x_description/meshes/link3.STL
- link link4: mass 0.38 -> 0.10451; geometry collision mesh filename=package://piper_x_description/meshes/link4.STL; visual mesh filename=package://piper_x_description/meshes/link4.STL
- link link5: mass 0.383 -> 0.053458; geometry collision mesh filename=package://piper_x_description/meshes/link5.STL; visual mesh filename=package://piper_x_description/meshes/link5.STL
- link link6: mass 0.007 -> 0.0061311; geometry collision mesh filename=package://piper_x_description/meshes/link6.STL; visual mesh filename=package://piper_x_description/meshes/link6.STL
Joints:
- joint joint1: axis 0 0 1 -> 0 -1 0; limit lower=-2.618 upper=2.168 effort=100 velocity=5 -> lower=-2.618 upper=2.618 effort=100 velocity=10; origin xyz=0 0 0.123 rpy=0 0 0 -> xyz=-0.00235357845905044 0.000777928765553683 0.119 rpy=1.5707963267949 0 0
- joint joint2: axis 0 0 1 -> 0 0 -1; limit lower=0 upper=3.14 effort=100 velocity=5 -> lower=0 upper=3.14 effort=100 velocity=10; origin xyz=0 0 0 rpy=1.5708 -0.10095 -3.1416 -> xyz=0 0 0 rpy=0 0 0
- joint joint3: limit lower=-2.967 upper=0 effort=100 velocity=5 -> lower=-2.9671 upper=0 effort=100 velocity=10; origin xyz=0.28503 0 0 rpy=0 0 -1.759 -> xyz=-0.2828 0.035596 0 rpy=3.1416 0 0
- joint joint4: axis 0 0 1 -> -0.15319 0 0.9882; limit lower=-1.745 upper=1.745 effort=100 velocity=5 -> lower=-1.57 upper=1.57 effort=100 velocity=10; origin xyz=-0.021984 -0.25075 0 rpy=1.5708 0 0 -> xyz=0.2693 -0.048542 -0.0042488 rpy=1.5708 0 1.5708
- joint joint5: limit lower=-1.22 upper=1.22 effort=100 velocity=5 -> lower=-1.57 upper=1.57 effort=100 velocity=10; origin xyz=0 0 0 rpy=-1.5708 0 0 -> xyz=-0.0071013 0.0034704 0.072275 rpy=0 -1.4729 -3.1416
- joint joint6: axis 0 0 1 -> 0.097757 0 -0.99521; limit lower=-2.0944 upper=2.0944 effort=100 velocity=3 -> lower=-3.14 upper=3.14 effort=100 velocity=10; origin xyz=8.8259E-05 -0.091 0 rpy=1.5708 0 0 -> xyz=0.0393 0 0 rpy=0 -1.4729 3.1416

Commit message: 🐞 fix(piper_description/urdf): 修正joint1的upper limit

File: src/piper_description/urdf/piper_description.urdf (robot description, URDF)
Before this commit: robot piper, 10 links, 9 joints
Joints:
- joint joint1: limit lower=-2.618 upper=2.168 effort=100 velocity=5 -> lower=-2.618 upper=2.618 effort=100 velocity=5

File: src/piper_description/urdf/piper_description.xacro (robot description, xacro)
@@ -86,5 +86,5 @@
     <limit
       lower="-2.618"
-      upper="2.168"
+      upper="2.618"
       effort="100"
       velocity="5" />

File: src/piper_description/urdf/piper_description_gazebo.xacro (robot description, xacro)
@@ -86,5 +86,5 @@
     <limit
       lower="-2.618"
-      upper="2.168"
+      upper="2.618"
       effort="100"
       velocity="5" />

File: src/piper_description/urdf/piper_description_old.urdf (robot description, URDF)
Before this commit: robot piper, 10 links, 9 joints
Joints:
- joint joint1: limit lower=-2.618 upper=2.168 effort=100 velocity=5 -> lower=-2.618 upper=2.618 effort=100 velocity=5

File: src/piper_description/urdf/piper_no_gripper_description.urdf (robot description, URDF)
Before this commit: robot piper, 7 links, 6 joints
Joints:
- joint joint1: limit lower=-2.618 upper=2.168 effort=100 velocity=5 -> lower=-2.618 upper=2.618 effort=100 velocity=5

File: src/piper_description/urdf/piper_no_gripper_description.xacro (robot description, xacro)
@@ -86,5 +86,5 @@
     <limit
       lower="-2.618"
-      upper="2.168"
+      upper="2.618"
       effort="100"
       velocity="5" />

File: src/piper_description/urdf/piper_no_gripper_description_gazebo.xacro (robot description, xacro)
@@ -86,5 +86,5 @@
     <limit
       lower="-2.618"
-      upper="2.168"
+      upper="2.618"
       effort="100"
       velocity="5" />

File: src/piper_description/urdf/piper_no_gripper_description_old.urdf (robot description, URDF)
Before this commit: robot piper, 7 links, 6 joints
Joints:
- joint joint1: limit lower=-2.618 upper=2.168 effort=100 velocity=5 -> lower=-2.618 upper=2.618 effort=100 velocity=5
