Commit message: ✨ feat(urdf, moveit): 修改urdf; 修改moveit下发的joint_states频率
修改urdf文件的重心和惯性张量；降低moveit的joint_states频率为200hz；修改mujoco部分readme

File: src/piper_description/urdf/piper_description.urdf (robot description, URDF)
Before this commit: robot piper, 10 links, 9 joints
Links:
- link link2: mass 1.17 -> 1.16
- link link5: mass 0.383 -> 0.39
- link link6: mass 0.00699089613564366 -> 0.46

File: src/piper_description/urdf/piper_description.xacro (robot description, xacro)
@@ -44,7 +44,7 @@
     name="link1">
     <inertial>
-            <origin xyz="0.000121504734057468 0.000104632162460536 -0.00438597309559853" rpy="0 0 0" />
-            <mass value="0.71" />
-            <inertia ixx="0.00048916" ixy="-0.00000036" ixz="-0.00000224" iyy="0.00040472" iyz="-0.00000242" izz="0.00043982" />
+      <origin xyz="0.00032 -0.00041 -0.00348" rpy="0 0 0" />
+      <mass value="0.71" />
+      <inertia ixx="0.00050027" ixy="0.00000078" ixz="0.00000626" iyy="0.00040879" iyz="0.00000462" izz="0.00045802" />
     </inertial>
     <visual>
@@ -93,7 +93,7 @@
     name="link2">
     <inertial>
-            <origin xyz="0.198666145229743 -0.010926924140076 0.00142121714502687" rpy="0 0 0" />
-            <mass value="1.17" />
-            <inertia ixx="0.00116918" ixy="-0.00180037" ixz="0.00025146" iyy="0.06785384" iyz="-0.00000455" izz="0.06774489" />
+      <origin xyz="0.21852 -0.00861 0.00126" rpy="0 0 0" />
+      <mass value="1.16" />
+      <inertia ixx="0.00111915" ixy="0.00182916" ixz="0.00019233" iyy="0.06763251" iyz="0.00000767" izz="0.067559" />
     </inertial>
     <visual>
@@ -143,7 +143,7 @@
     name="link3">
     <inertial>
-            <origin xyz="-0.0202737662122021 -0.133914995944595 -0.000458682652737356" rpy="0 0 0" />
-            <mass value="0.5" />
-            <inertia ixx="0.01361711" ixy="0.00165794" ixz="-0.00000048" iyy="0.00045024" iyz="-0.00000045" izz="0.01380322" />
+      <origin xyz="-0.01999 -0.14808 -0.00053" rpy="0 0 0" />
+      <mass value="0.5" />
+      <inertia ixx="0.01347608" ixy="0.00161034" ixz="0.00000066" iyy="0.00046377" iyz="0.00000162" izz="0.01363321" />
     </inertial>
     <visual>
@@ -193,7 +193,7 @@
     name="link4">
     <inertial>
-            <origin xyz="-9.66635791618542E-05 0.000876064475651083 -0.00496880904640868" rpy="0 0 0" />
-            <mass value="0.38" />
-            <inertia ixx="0.00018501" ixy="0.00000054" ixz="0.00000120" iyy="0.00018965" iyz="-0.00000841" izz="0.00015484" />
+      <origin xyz="0.00013 -0.00076 -0.00394" rpy="0 0 0" />
+      <mass value="0.38" />
+      <inertia ixx="0.00017844" ixy="0.00000062" ixz="0.00000067" iyy="0.00018914" iyz="0.00000408" izz="0.00014613" />
     </inertial>
     <visual>
@@ -242,7 +242,7 @@
     name="link5">
     <inertial>
-            <origin xyz="-4.10554118924211E-05 -0.0566486692356075 -0.0037205791677906" rpy="0 0 0" />
-            <mass value="0.383" />
-            <inertia ixx="0.00166169" ixy="0.00000006" ixz="-0.00000007" iyy="0.00018510" iyz="0.00001026" izz="0.00164321" />
+      <origin xyz="0.00018 -0.06104 -0.00227" rpy="0 0 0" />
+      <mass value="0.39" />
+      <inertia ixx="0.00172318" ixy="0.00000259" ixz="0.00000010" iyy="0.00017936" iyz="0.00000990" izz="0.00171172" />
     </inertial>
     <visual>
@@ -291,7 +291,7 @@
     name="link6">
     <inertial>
-            <origin xyz="-8.82590762930069E-05 9.0598378529832E-06 -0.002" rpy="0 0 0" />
-            <mass value="0.00699089613564366" />
-            <inertia ixx="5.73015540542155E-07" ixy="-1.98305403089247E-22" ixz="-7.2791893904596E-23" iyy="5.73015540542155E-07" iyz="-3.4146026640245E-24" izz="1.06738869138926E-06" />
+      <origin xyz="-0.00003 0.00006 0.04618" rpy="0 0 0" />
+      <mass value="0.46" />
+      <inertia ixx="0.00152112" ixy="0.00000202" ixz="0.00000261" iyy="0.00138626" iyz="0.00000002" izz="0.00031152" />
     </inertial>
     <visual>

File: src/piper_description/urdf/piper_description_gazebo.xacro (robot description, xacro)
@@ -44,7 +44,7 @@
     name="link1">
     <inertial>
-            <origin xyz="0.000121504734057468 0.000104632162460536 -0.00438597309559853" rpy="0 0 0" />
-            <mass value="0.71" />
-            <inertia ixx="0.00048916" ixy="-0.00000036" ixz="-0.00000224" iyy="0.00040472" iyz="-0.00000242" izz="0.00043982" />
+      <origin xyz="0.00032 -0.00041 -0.00348" rpy="0 0 0" />
+      <mass value="0.71" />
+      <inertia ixx="0.00050027" ixy="0.00000078" ixz="0.00000626" iyy="0.00040879" iyz="0.00000462" izz="0.00045802" />
     </inertial>
     <visual>
@@ -93,7 +93,7 @@
     name="link2">
     <inertial>
-            <origin xyz="0.198666145229743 -0.010926924140076 0.00142121714502687" rpy="0 0 0" />
-            <mass value="1.17" />
-            <inertia ixx="0.00116918" ixy="-0.00180037" ixz="0.00025146" iyy="0.06785384" iyz="-0.00000455" izz="0.06774489" />
+      <origin xyz="0.21852 -0.00861 0.00126" rpy="0 0 0" />
+      <mass value="1.16" />
+      <inertia ixx="0.00111915" ixy="0.00182916" ixz="0.00019233" iyy="0.06763251" iyz="0.00000767" izz="0.067559" />
     </inertial>
     <visual>
@@ -143,7 +143,7 @@
     name="link3">
     <inertial>
-            <origin xyz="-0.0202737662122021 -0.133914995944595 -0.000458682652737356" rpy="0 0 0" />
-            <mass value="0.5" />
-            <inertia ixx="0.01361711" ixy="0.00165794" ixz="-0.00000048" iyy="0.00045024" iyz="-0.00000045" izz="0.01380322" />
+      <origin xyz="-0.01999 -0.14808 -0.00053" rpy="0 0 0" />
+      <mass value="0.5" />
+      <inertia ixx="0.01347608" ixy="0.00161034" ixz="0.00000066" iyy="0.00046377" iyz="0.00000162" izz="0.01363321" />
     </inertial>
     <visual>
@@ -193,7 +193,7 @@
     name="link4">
     <inertial>
-            <origin xyz="-9.66635791618542E-05 0.000876064475651083 -0.00496880904640868" rpy="0 0 0" />
-            <mass value="0.38" />
-            <inertia ixx="0.00018501" ixy="0.00000054" ixz="0.00000120" iyy="0.00018965" iyz="-0.00000841" izz="0.00015484" />
+      <origin xyz="0.00013 -0.00076 -0.00394" rpy="0 0 0" />
+      <mass value="0.38" />
+      <inertia ixx="0.00017844" ixy="0.00000062" ixz="0.00000067" iyy="0.00018914" iyz="0.00000408" izz="0.00014613" />
     </inertial>
     <visual>
@@ -242,7 +242,7 @@
     name="link5">
     <inertial>
-            <origin xyz="-4.10554118924211E-05 -0.0566486692356075 -0.0037205791677906" rpy="0 0 0" />
-            <mass value="0.383" />
-            <inertia ixx="0.00166169" ixy="0.00000006" ixz="-0.00000007" iyy="0.00018510" iyz="0.00001026" izz="0.00164321" />
+      <origin xyz="0.00018 -0.06104 -0.00227" rpy="0 0 0" />
+      <mass value="0.39" />
+      <inertia ixx="0.00172318" ixy="0.00000259" ixz="0.00000010" iyy="0.00017936" iyz="0.00000990" izz="0.00171172" />
     </inertial>
     <visual>
@@ -291,7 +291,7 @@
     name="link6">
     <inertial>
-            <origin xyz="-8.82590762930069E-05 9.0598378529832E-06 -0.002" rpy="0 0 0" />
-            <mass value="0.00699089613564366" />
-            <inertia ixx="5.73015540542155E-07" ixy="-1.98305403089247E-22" ixz="-7.2791893904596E-23" iyy="5.73015540542155E-07" iyz="-3.4146026640245E-24" izz="1.06738869138926E-06" />
+      <origin xyz="-0.00003 0.00006 0.04618" rpy="0 0 0" />
+      <mass value="0.46" />
+      <inertia ixx="0.00152112" ixy="0.00000202" ixz="0.00000261" iyy="0.00138626" iyz="0.00000002" izz="0.00031152" />
     </inertial>
     <visual>

File: src/piper_description/urdf/piper_description_old.urdf (robot description, URDF)
Before this commit: robot piper, 10 links, 9 joints
Links:
- link link2: mass 1.17 -> 1.16
- link link5: mass 0.383 -> 0.39
- link link6: mass 0.00699089613564366 -> 0.46

File: src/piper_description/urdf/piper_no_gripper_description.urdf (robot description, URDF)
Before this commit: robot piper, 7 links, 6 joints
Links:
- link link2: mass 1.17 -> 1.16
- link link5: mass 0.383 -> 0.39
- link link6: mass 0.00699089613564366 -> 0.46

File: src/piper_description/urdf/piper_no_gripper_description.xacro (robot description, xacro)
@@ -44,7 +44,7 @@
     name="link1">
     <inertial>
-            <origin xyz="0.000121504734057468 0.000104632162460536 -0.00438597309559853" rpy="0 0 0" />
-            <mass value="0.71" />
-            <inertia ixx="0.00048916" ixy="-0.00000036" ixz="-0.00000224" iyy="0.00040472" iyz="-0.00000242" izz="0.00043982" />
+      <origin xyz="0.00032 -0.00041 -0.00348" rpy="0 0 0" />
+      <mass value="0.71" />
+      <inertia ixx="0.00050027" ixy="0.00000078" ixz="0.00000626" iyy="0.00040879" iyz="0.00000462" izz="0.00045802" />
     </inertial>
     <visual>
@@ -93,7 +93,7 @@
     name="link2">
     <inertial>
-      <origin xyz="0.198666145229743 -0.010926924140076 0.00142121714502687" rpy="0 0 0" />
-      <mass value="1.17" />
-      <inertia ixx="0.00116918" ixy="-0.00180037" ixz="0.00025146" iyy="0.06785384" iyz="-0.00000455" izz="0.06774489" />
+      <origin xyz="0.21852 -0.00861 0.00126" rpy="0 0 0" />
+      <mass value="1.16" />
+      <inertia ixx="0.00111915" ixy="0.00182916" ixz="0.00019233" iyy="0.06763251" iyz="0.00000767" izz="0.067559" />
     </inertial>
     <visual>
@@ -143,7 +143,7 @@
     name="link3">
     <inertial>
-      <origin xyz="-0.0202737662122021 -0.133914995944595 -0.000458682652737356" rpy="0 0 0" />
+      <origin xyz="-0.01999 -0.14808 -0.00053" rpy="0 0 0" />
       <mass value="0.5" />
-      <inertia ixx="0.01361711" ixy="0.00165794" ixz="-0.00000048" iyy="0.00045024" iyz="-0.00000045" izz="0.01380322" />
+      <inertia ixx="0.01347608" ixy="0.00161034" ixz="0.00000066" iyy="0.00046377" iyz="0.00000162" izz="0.01363321" />
     </inertial>
     <visual>
@@ -193,7 +193,7 @@
     name="link4">
     <inertial>
-      <origin xyz="-9.66635791618542E-05 0.000876064475651083 -0.00496880904640868" rpy="0 0 0" />
+      <origin xyz="0.00013 -0.00076 -0.00394" rpy="0 0 0" />
       <mass value="0.38" />
-      <inertia ixx="0.00018501" ixy="0.00000054" ixz="0.00000120" iyy="0.00018965" iyz="-0.00000841" izz="0.00015484" />
+      <inertia ixx="0.00017844" ixy="0.00000062" ixz="0.00000067" iyy="0.00018914" iyz="0.00000408" izz="0.00014613" />
     </inertial>
     <visual>
@@ -242,7 +242,7 @@
     name="link5">
     <inertial>
-      <origin xyz="-4.10554118924211E-05 -0.0566486692356075 -0.0037205791677906" rpy="0 0 0" />
-      <mass value="0.383" />
-      <inertia ixx="0.00166169" ixy="0.00000006" ixz="-0.00000007" iyy="0.00018510" iyz="0.00001026" izz="0.00164321" />
+      <origin xyz="0.00018 -0.06104 -0.00227" rpy="0 0 0" />
+      <mass value="0.39" />
+      <inertia ixx="0.00172318" ixy="0.00000259" ixz="0.00000010" iyy="0.00017936" iyz="0.00000990" izz="0.00171172" />
     </inertial>
     <visual>
@@ -291,7 +291,7 @@
     name="link6">
     <inertial>
-      <origin xyz="-8.82590762930069E-05 9.0598378529832E-06 -0.002" rpy="0 0 0" />
-      <mass value="0.00699089613564366" />
-      <inertia ixx="5.73015540542155E-07" ixy="-1.98305403089247E-22" ixz="-7.2791893904596E-23" iyy="5.73015540542155E-07" iyz="-3.4146026640245E-24" izz="1.06738869138926E-06" />
+      <origin xyz="-0.00003 0.00006 0.04618" rpy="0 0 0" />
+      <mass value="0.46" />
+      <inertia ixx="0.00152112" ixy="0.00000202" ixz="0.00000261" iyy="0.00138626" iyz="0.00000002" izz="0.00031152" />
     </inertial>
     <visual>

File: src/piper_description/urdf/piper_no_gripper_description_gazebo.xacro (robot description, xacro)
@@ -44,7 +44,7 @@
     name="link1">
     <inertial>
-            <origin xyz="0.000121504734057468 0.000104632162460536 -0.00438597309559853" rpy="0 0 0" />
-            <mass value="0.71" />
-            <inertia ixx="0.00048916" ixy="-0.00000036" ixz="-0.00000224" iyy="0.00040472" iyz="-0.00000242" izz="0.00043982" />
+      <origin xyz="0.00032 -0.00041 -0.00348" rpy="0 0 0" />
+      <mass value="0.71" />
+      <inertia ixx="0.00050027" ixy="0.00000078" ixz="0.00000626" iyy="0.00040879" iyz="0.00000462" izz="0.00045802" />
     </inertial>
     <visual>
@@ -93,7 +93,7 @@
     name="link2">
     <inertial>
-            <origin xyz="0.198666145229743 -0.010926924140076 0.00142121714502687" rpy="0 0 0" />
-            <mass value="1.17" />
-            <inertia ixx="0.00116918" ixy="-0.00180037" ixz="0.00025146" iyy="0.06785384" iyz="-0.00000455" izz="0.06774489" />
+      <origin xyz="0.21852 -0.00861 0.00126" rpy="0 0 0" />
+      <mass value="1.16" />
+      <inertia ixx="0.00111915" ixy="0.00182916" ixz="0.00019233" iyy="0.06763251" iyz="0.00000767" izz="0.067559" />
     </inertial>
     <visual>
@@ -143,7 +143,7 @@
     name="link3">
     <inertial>
-            <origin xyz="-0.0202737662122021 -0.133914995944595 -0.000458682652737356" rpy="0 0 0" />
-            <mass value="0.5" />
-            <inertia ixx="0.01361711" ixy="0.00165794" ixz="-0.00000048" iyy="0.00045024" iyz="-0.00000045" izz="0.01380322" />
+      <origin xyz="-0.01999 -0.14808 -0.00053" rpy="0 0 0" />
+      <mass value="0.5" />
+      <inertia ixx="0.01347608" ixy="0.00161034" ixz="0.00000066" iyy="0.00046377" iyz="0.00000162" izz="0.01363321" />
     </inertial>
     <visual>
@@ -193,7 +193,7 @@
     name="link4">
     <inertial>
-            <origin xyz="-9.66635791618542E-05 0.000876064475651083 -0.00496880904640868" rpy="0 0 0" />
-            <mass value="0.38" />
-            <inertia ixx="0.00018501" ixy="0.00000054" ixz="0.00000120" iyy="0.00018965" iyz="-0.00000841" izz="0.00015484" />
+      <origin xyz="0.00013 -0.00076 -0.00394" rpy="0 0 0" />
+      <mass value="0.38" />
+      <inertia ixx="0.00017844" ixy="0.00000062" ixz="0.00000067" iyy="0.00018914" iyz="0.00000408" izz="0.00014613" />
     </inertial>
     <visual>
@@ -242,7 +242,7 @@
     name="link5">
     <inertial>
-            <origin xyz="-4.10554118924211E-05 -0.0566486692356075 -0.0037205791677906" rpy="0 0 0" />
-            <mass value="0.383" />
-            <inertia ixx="0.00166169" ixy="0.00000006" ixz="-0.00000007" iyy="0.00018510" iyz="0.00001026" izz="0.00164321" />
+      <origin xyz="0.00018 -0.06104 -0.00227" rpy="0 0 0" />
+      <mass value="0.39" />
+      <inertia ixx="0.00172318" ixy="0.00000259" ixz="0.00000010" iyy="0.00017936" iyz="0.00000990" izz="0.00171172" />
     </inertial>
     <visual>
@@ -291,7 +291,7 @@
     name="link6">
     <inertial>
-            <origin xyz="-8.82590762930069E-05 9.0598378529832E-06 -0.002" rpy="0 0 0" />
-            <mass value="0.00699089613564366" />
-            <inertia ixx="5.73015540542155E-07" ixy="-1.98305403089247E-22" ixz="-7.2791893904596E-23" iyy="5.73015540542155E-07" iyz="-3.4146026640245E-24" izz="1.06738869138926E-06" />
+      <origin xyz="-0.00003 0.00006 0.04618" rpy="0 0 0" />
+      <mass value="0.46" />
+      <inertia ixx="0.00152112" ixy="0.00000202" ixz="0.00000261" iyy="0.00138626" iyz="0.00000002" izz="0.00031152" />
     </inertial>
     <visual>

File: src/piper_description/urdf/piper_no_gripper_description_old.urdf (robot description, URDF)
Before this commit: robot piper, 7 links, 6 joints
Links:
- link link2: mass 1.17 -> 1.16
- link link5: mass 0.383 -> 0.39
- link link6: mass 0.00699089613564366 -> 0.46

Commit message: ✨ feat(urdf): 修改link5和link6的质量为0.383kg和0.007kg

File: src/piper_description/urdf/piper_description.urdf (robot description, URDF)
Before this commit: robot piper, 10 links, 9 joints
Links:
- link link5: mass 0.39 -> 0.383
- link link6: mass 0.46 -> 0.007

File: src/piper_description/urdf/piper_description.xacro (robot description, xacro)
@@ -243,5 +243,5 @@
     <inertial>
       <origin xyz="0.00018 -0.06104 -0.00227" rpy="0 0 0" />
-      <mass value="0.39" />
+      <mass value="0.383" />
       <inertia ixx="0.00172318" ixy="0.00000259" ixz="0.00000010" iyy="0.00017936" iyz="0.00000990" izz="0.00171172" />
     </inertial>
@@ -292,5 +292,5 @@
     <inertial>
       <origin xyz="-0.00003 0.00006 0.04618" rpy="0 0 0" />
-      <mass value="0.46" />
+      <mass value="0.007" />
       <inertia ixx="0.00152112" ixy="0.00000202" ixz="0.00000261" iyy="0.00138626" iyz="0.00000002" izz="0.00031152" />
     </inertial>

File: src/piper_description/urdf/piper_description_gazebo.xacro (robot description, xacro)
@@ -243,5 +243,5 @@
     <inertial>
       <origin xyz="0.00018 -0.06104 -0.00227" rpy="0 0 0" />
-      <mass value="0.39" />
+      <mass value="0.383" />
       <inertia ixx="0.00172318" ixy="0.00000259" ixz="0.00000010" iyy="0.00017936" iyz="0.00000990" izz="0.00171172" />
     </inertial>
@@ -292,5 +292,5 @@
     <inertial>
       <origin xyz="-0.00003 0.00006 0.04618" rpy="0 0 0" />
-      <mass value="0.46" />
+      <mass value="0.007" />
       <inertia ixx="0.00152112" ixy="0.00000202" ixz="0.00000261" iyy="0.00138626" iyz="0.00000002" izz="0.00031152" />
     </inertial>

File: src/piper_description/urdf/piper_description_old.urdf (robot description, URDF)
Before this commit: robot piper, 10 links, 9 joints
Links:
- link link5: mass 0.39 -> 0.383
- link link6: mass 0.46 -> 0.007

File: src/piper_description/urdf/piper_description_with_teach.urdf (robot description, URDF)
Before this commit: robot piper, 10 links, 9 joints
Links:
- link link5: mass 0.39 -> 0.383
- link link6: mass 0.46 -> 0.007

File: src/piper_description/urdf/piper_no_gripper_description.urdf (robot description, URDF)
Before this commit: robot piper, 7 links, 6 joints
Links:
- link link5: mass 0.39 -> 0.383
- link link6: mass 0.46 -> 0.007

File: src/piper_description/urdf/piper_no_gripper_description.xacro (robot description, xacro)
@@ -243,5 +243,5 @@
     <inertial>
       <origin xyz="0.00018 -0.06104 -0.00227" rpy="0 0 0" />
-      <mass value="0.39" />
+      <mass value="0.383" />
       <inertia ixx="0.00172318" ixy="0.00000259" ixz="0.00000010" iyy="0.00017936" iyz="0.00000990" izz="0.00171172" />
     </inertial>
@@ -292,5 +292,5 @@
     <inertial>
       <origin xyz="-0.00003 0.00006 0.04618" rpy="0 0 0" />
-      <mass value="0.46" />
+      <mass value="0.007" />
       <inertia ixx="0.00152112" ixy="0.00000202" ixz="0.00000261" iyy="0.00138626" iyz="0.00000002" izz="0.00031152" />
     </inertial>

File: src/piper_description/urdf/piper_no_gripper_description_gazebo.xacro (robot description, xacro)
@@ -243,5 +243,5 @@
     <inertial>
       <origin xyz="0.00018 -0.06104 -0.00227" rpy="0 0 0" />
-      <mass value="0.39" />
+      <mass value="0.383" />
       <inertia ixx="0.00172318" ixy="0.00000259" ixz="0.00000010" iyy="0.00017936" iyz="0.00000990" izz="0.00171172" />
     </inertial>
@@ -292,5 +292,5 @@
     <inertial>
       <origin xyz="-0.00003 0.00006 0.04618" rpy="0 0 0" />
-      <mass value="0.46" />
+      <mass value="0.007" />
       <inertia ixx="0.00152112" ixy="0.00000202" ixz="0.00000261" iyy="0.00138626" iyz="0.00000002" izz="0.00031152" />
     </inertial>

File: src/piper_description/urdf/piper_no_gripper_description_old.urdf (robot description, URDF)
Before this commit: robot piper, 7 links, 6 joints
Links:
- link link5: mass 0.39 -> 0.383
- link link6: mass 0.46 -> 0.007

Commit message: setups at 25/2

File: src/piper_description/urdf/piper_description.urdf (robot description, URDF)
Before this commit: robot piper, 10 links, 9 joints
Links:
- added link camera_link, mass 0.0067926; collision box size=0.001 0.001 0.001; visual box size=0.02 0.05 0.02
Joints:
- added joint hand_camera_joint: type fixed, parent link6, child camera_link, origin xyz=0.07 0.0 0.0 rpy=0.0 -1.57 0.0, axis 0 0 0

File: src/piper_description/urdf/piper_description.xacro (robot description, xacro)
@@ -332,6 +332,6 @@
       xyz="0 0 1" />
     <limit
-      lower="-2.0944"
-      upper="2.0944"
+      lower="0.0"
+      upper="3.14159"
       effort="100"
       velocity="3" />
@@ -503,4 +503,55 @@
       effort="10"
       velocity="1" />
+  </joint>
+  <link
+    name="camera_link">
+    <inertial>
+      <origin
+        xyz="0.0 0.0 0.0"
+        rpy="0 0 0" />
+      <mass
+        value="0.0067926" />
+      <inertia
+        ixx="3.7811E-05"
+        ixy="2.2861E-18"
+        ixz="2.2446E-19"
+        iyy="9.4061E-05"
+        iyz="6.1172E-06"
+        izz="0.00012345" />
+    </inertial>
+    <visual>
+      <origin
+        xyz="0 0 0"
+        rpy="0 0 0" />
+      <geometry>
+          <box size="0.02 0.05 0.02"/>
+      </geometry>
+      <material
+        name="">
+        <color
+          rgba="1 1 1 1" />
+      </material>
+    </visual>
+    <collision>
+      <origin
+        xyz="0 0 0"
+        rpy="0 1.57 0" />
+      <geometry>
+        <box size="0.001 0.001 0.001"/>
+      </geometry>
+    </collision>
+  </link>
+  <joint
+    name="hand_camera_joint"
+    type="fixed">
+    <origin
+      xyz="0.07 0.0 0.0"
+      rpy="0.0 -1.57 0.0" />
+    <parent
+      link="link6" />
+    <child
+      link="camera_link" />
+    <axis
+      xyz="0 0 0" />
   </joint>
 <!-- controller -->
