Commit message: update piper x pkg name

File: src/piper_x_description/urdf/piper_x_description.urdf (robot description, URDF)
Before this commit: robot piper_x_description_v3, 9 links, 8 joints
Links:
- link Link1: geometry collision mesh filename=package://piper_x_description/meshes/dae/J1.dae; visual mesh filename=package://piper_x_description/meshes/dae/J1.dae
- link Link2: geometry collision mesh filename=package://piper_x_description/meshes/dae/J2.dae; visual mesh filename=package://piper_x_description/meshes/dae/J2.dae
- link Link3: geometry collision mesh filename=package://piper_x_description/meshes/dae/J3.dae; visual mesh filename=package://piper_x_description/meshes/dae/J3.dae
- link Link4: geometry collision mesh filename=package://piper_x_description/meshes/dae/J4.dae; visual mesh filename=package://piper_x_description/meshes/dae/J4.dae
- link Link5: geometry collision mesh filename=package://piper_x_description/meshes/dae/J5.dae; visual mesh filename=package://piper_x_description/meshes/dae/J5.dae
- link Link6: geometry collision mesh filename=package://piper_x_description/meshes/dae/gripper_base_100_v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 scale=0.8 0.8 0.8; visual mesh filename=package://piper_x_description/meshes/dae/gripper_base_100_v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 scale=0.8 0.8 0.8
- link Link7: geometry collision mesh filename=package://piper_x_description/meshes/dae/J7.dae; visual mesh filename=package://piper_x_description/meshes/dae/J7.dae
- link Link8: geometry collision mesh filename=package://piper_x_description/meshes/dae/J8.dae; visual mesh filename=package://piper_x_description/meshes/dae/J8.dae
- link base_link: geometry collision mesh filename=package://piper_x_description/meshes/dae/base_Link.dae; visual mesh filename=package://piper_x_description/meshes/dae/base_Link.dae
