Commit message: ad增加piper urdf 深色版本，用于适配isaac sim

File: src/robot_description/piper_description/urdf/piper_description.urdf (robot description, URDF)
Before this commit: robot piper, 10 links, 9 joints
Links:
- link link2: mass 1.16 -> 1.17
- link link6: mass 0.007 -> 0.00699089613564366
Joints:
- joint joint1: limit lower=-2.618 upper=2.618 effort=100 velocity=5 -> lower=-2.618 upper=2.168 effort=100 velocity=5

File: src/robot_description/piper_description/urdf/piper_description.xacro (robot description, xacro)
@@ -44,7 +44,7 @@
     name="link1">
     <inertial>
-      <origin xyz="0.00032 -0.00041 -0.00348" rpy="0 0 0" />
-      <mass value="0.71" />
-      <inertia ixx="0.00050027" ixy="0.00000078" ixz="0.00000626" iyy="0.00040879" iyz="0.00000462" izz="0.00045802" />
+            <origin xyz="0.000121504734057468 0.000104632162460536 -0.00438597309559853" rpy="0 0 0" />
+            <mass value="0.71" />
+            <inertia ixx="0.00048916" ixy="-0.00000036" ixz="-0.00000224" iyy="0.00040472" iyz="-0.00000242" izz="0.00043982" />
     </inertial>
     <visual>
@@ -86,5 +86,5 @@
     <limit
       lower="-2.618"
-      upper="2.618"
+      upper="2.168"
       effort="100"
       velocity="5" />
@@ -93,7 +93,7 @@
     name="link2">
     <inertial>
-      <origin xyz="0.21852 -0.00861 0.00126" rpy="0 0 0" />
-      <mass value="1.16" />
-      <inertia ixx="0.00111915" ixy="0.00182916" ixz="0.00019233" iyy="0.06763251" iyz="0.00000767" izz="0.067559" />
+            <origin xyz="0.198666145229743 -0.010926924140076 0.00142121714502687" rpy="0 0 0" />
+            <mass value="1.17" />
+            <inertia ixx="0.00116918" ixy="-0.00180037" ixz="0.00025146" iyy="0.06785384" iyz="-0.00000455" izz="0.06774489" />
     </inertial>
     <visual>
@@ -143,7 +143,7 @@
     name="link3">
     <inertial>
-      <origin xyz="-0.01999 -0.14808 -0.00053" rpy="0 0 0" />
-      <mass value="0.5" />
-      <inertia ixx="0.01347608" ixy="0.00161034" ixz="0.00000066" iyy="0.00046377" iyz="0.00000162" izz="0.01363321" />
+            <origin xyz="-0.0202737662122021 -0.133914995944595 -0.000458682652737356" rpy="0 0 0" />
+            <mass value="0.5" />
+            <inertia ixx="0.01361711" ixy="0.00165794" ixz="-0.00000048" iyy="0.00045024" iyz="-0.00000045" izz="0.01380322" />
     </inertial>
     <visual>
@@ -193,7 +193,7 @@
     name="link4">
     <inertial>
-      <origin xyz="0.00013 -0.00076 -0.00394" rpy="0 0 0" />
-      <mass value="0.38" />
-      <inertia ixx="0.00017844" ixy="0.00000062" ixz="0.00000067" iyy="0.00018914" iyz="0.00000408" izz="0.00014613" />
+            <origin xyz="-9.66635791618542E-05 0.000876064475651083 -0.00496880904640868" rpy="0 0 0" />
+            <mass value="0.38" />
+            <inertia ixx="0.00018501" ixy="0.00000054" ixz="0.00000120" iyy="0.00018965" iyz="-0.00000841" izz="0.00015484" />
     </inertial>
     <visual>
@@ -242,7 +242,7 @@
     name="link5">
     <inertial>
-      <origin xyz="0.00018 -0.06104 -0.00227" rpy="0 0 0" />
-      <mass value="0.383" />
-      <inertia ixx="0.00172318" ixy="0.00000259" ixz="0.00000010" iyy="0.00017936" iyz="0.00000990" izz="0.00171172" />
+            <origin xyz="-4.10554118924211E-05 -0.0566486692356075 -0.0037205791677906" rpy="0 0 0" />
+            <mass value="0.383" />
+            <inertia ixx="0.00166169" ixy="0.00000006" ixz="-0.00000007" iyy="0.00018510" iyz="0.00001026" izz="0.00164321" />
     </inertial>
     <visual>
@@ -291,7 +291,7 @@
     name="link6">
     <inertial>
-      <origin xyz="-0.00003 0.00006 0.04618" rpy="0 0 0" />
-      <mass value="0.007" />
-      <inertia ixx="0.00152112" ixy="0.00000202" ixz="0.00000261" iyy="0.00138626" iyz="0.00000002" izz="0.00031152" />
+            <origin xyz="-8.82590762930069E-05 9.0598378529832E-06 -0.002" rpy="0 0 0" />
+            <mass value="0.00699089613564366" />
+            <inertia ixx="5.73015540542155E-07" ixy="-1.98305403089247E-22" ixz="-7.2791893904596E-23" iyy="5.73015540542155E-07" iyz="-3.4146026640245E-24" izz="1.06738869138926E-06" />
     </inertial>
     <visual>
@@ -400,5 +400,5 @@
         ixy="-0.00000113"
         ixz="0.00000021"
-        iyy="0.00000781"
+        iyy="-0.00000113"
         iyz="-0.00001372"
         izz="0.0000747" />
@@ -458,5 +458,5 @@
         ixy="-0.00000113"
         ixz="0.00000021"
-        iyy="0.00000781"
+        iyy="-0.00000113"
         iyz="-0.00001372"
         izz="0.0000747" />

File: src/robot_description/piper_description/urdf/piper_description_gazebo.xacro (robot description, xacro)
@@ -44,7 +44,7 @@
     name="link1">
     <inertial>
-      <origin xyz="0.00032 -0.00041 -0.00348" rpy="0 0 0" />
-      <mass value="0.71" />
-      <inertia ixx="0.00050027" ixy="0.00000078" ixz="0.00000626" iyy="0.00040879" iyz="0.00000462" izz="0.00045802" />
+            <origin xyz="0.000121504734057468 0.000104632162460536 -0.00438597309559853" rpy="0 0 0" />
+            <mass value="0.71" />
+            <inertia ixx="0.00048916" ixy="-0.00000036" ixz="-0.00000224" iyy="0.00040472" iyz="-0.00000242" izz="0.00043982" />
     </inertial>
     <visual>
@@ -86,5 +86,5 @@
     <limit
       lower="-2.618"
-      upper="2.618"
+      upper="2.168"
       effort="100"
       velocity="5" />
@@ -93,7 +93,7 @@
     name="link2">
     <inertial>
-      <origin xyz="0.21852 -0.00861 0.00126" rpy="0 0 0" />
-      <mass value="1.16" />
-      <inertia ixx="0.00111915" ixy="0.00182916" ixz="0.00019233" iyy="0.06763251" iyz="0.00000767" izz="0.067559" />
+            <origin xyz="0.198666145229743 -0.010926924140076 0.00142121714502687" rpy="0 0 0" />
+            <mass value="1.17" />
+            <inertia ixx="0.00116918" ixy="-0.00180037" ixz="0.00025146" iyy="0.06785384" iyz="-0.00000455" izz="0.06774489" />
     </inertial>
     <visual>
@@ -143,7 +143,7 @@
     name="link3">
     <inertial>
-      <origin xyz="-0.01999 -0.14808 -0.00053" rpy="0 0 0" />
-      <mass value="0.5" />
-      <inertia ixx="0.01347608" ixy="0.00161034" ixz="0.00000066" iyy="0.00046377" iyz="0.00000162" izz="0.01363321" />
+            <origin xyz="-0.0202737662122021 -0.133914995944595 -0.000458682652737356" rpy="0 0 0" />
+            <mass value="0.5" />
+            <inertia ixx="0.01361711" ixy="0.00165794" ixz="-0.00000048" iyy="0.00045024" iyz="-0.00000045" izz="0.01380322" />
     </inertial>
     <visual>
@@ -193,7 +193,7 @@
     name="link4">
     <inertial>
-      <origin xyz="0.00013 -0.00076 -0.00394" rpy="0 0 0" />
-      <mass value="0.38" />
-      <inertia ixx="0.00017844" ixy="0.00000062" ixz="0.00000067" iyy="0.00018914" iyz="0.00000408" izz="0.00014613" />
+            <origin xyz="-9.66635791618542E-05 0.000876064475651083 -0.00496880904640868" rpy="0 0 0" />
+            <mass value="0.38" />
+            <inertia ixx="0.00018501" ixy="0.00000054" ixz="0.00000120" iyy="0.00018965" iyz="-0.00000841" izz="0.00015484" />
     </inertial>
     <visual>
@@ -242,7 +242,7 @@
     name="link5">
     <inertial>
-      <origin xyz="0.00018 -0.06104 -0.00227" rpy="0 0 0" />
-      <mass value="0.383" />
-      <inertia ixx="0.00172318" ixy="0.00000259" ixz="0.00000010" iyy="0.00017936" iyz="0.00000990" izz="0.00171172" />
+            <origin xyz="-4.10554118924211E-05 -0.0566486692356075 -0.0037205791677906" rpy="0 0 0" />
+            <mass value="0.383" />
+            <inertia ixx="0.00166169" ixy="0.00000006" ixz="-0.00000007" iyy="0.00018510" iyz="0.00001026" izz="0.00164321" />
     </inertial>
     <visual>
@@ -291,7 +291,7 @@
     name="link6">
     <inertial>
-      <origin xyz="-0.00003 0.00006 0.04618" rpy="0 0 0" />
-      <mass value="0.007" />
-      <inertia ixx="0.00152112" ixy="0.00000202" ixz="0.00000261" iyy="0.00138626" iyz="0.00000002" izz="0.00031152" />
+            <origin xyz="-8.82590762930069E-05 9.0598378529832E-06 -0.002" rpy="0 0 0" />
+            <mass value="0.00699089613564366" />
+            <inertia ixx="5.73015540542155E-07" ixy="-1.98305403089247E-22" ixz="-7.2791893904596E-23" iyy="5.73015540542155E-07" iyz="-3.4146026640245E-24" izz="1.06738869138926E-06" />
     </inertial>
     <visual>
@@ -400,5 +400,5 @@
         ixy="-0.00000113"
         ixz="0.00000021"
-        iyy="0.00000781"
+        iyy="-0.00000113"
         iyz="-0.00001372"
         izz="0.0000747" />
@@ -458,5 +458,5 @@
         ixy="-0.00000113"
         ixz="0.00000021"
-        iyy="0.00000781"
+        iyy="-0.00000113"
         iyz="-0.00001372"
         izz="0.0000747" />

File: src/robot_description/piper_description/urdf/piper_description_old.urdf (robot description, URDF)
Before this commit: robot piper, 10 links, 9 joints
Links:
- link link2: mass 1.16 -> 1.17
- link link6: mass 0.007 -> 0.00699089613564366
Joints:
- joint joint1: limit lower=-2.618 upper=2.618 effort=100 velocity=5 -> lower=-2.618 upper=2.168 effort=100 velocity=5

File: src/robot_description/piper_description/urdf/piper_no_gripper_description.urdf (robot description, URDF)
Before this commit: robot piper, 7 links, 6 joints
Links:
- link link2: mass 1.16 -> 1.17
- link link6: mass 0.007 -> 0.00699089613564366
Joints:
- joint joint1: limit lower=-2.618 upper=2.618 effort=100 velocity=5 -> lower=-2.618 upper=2.168 effort=100 velocity=5

File: src/robot_description/piper_description/urdf/piper_no_gripper_description.xacro (robot description, xacro)
@@ -44,7 +44,7 @@
     name="link1">
     <inertial>
-      <origin xyz="0.00032 -0.00041 -0.00348" rpy="0 0 0" />
-      <mass value="0.71" />
-      <inertia ixx="0.00050027" ixy="0.00000078" ixz="0.00000626" iyy="0.00040879" iyz="0.00000462" izz="0.00045802" />
+            <origin xyz="0.000121504734057468 0.000104632162460536 -0.00438597309559853" rpy="0 0 0" />
+            <mass value="0.71" />
+            <inertia ixx="0.00048916" ixy="-0.00000036" ixz="-0.00000224" iyy="0.00040472" iyz="-0.00000242" izz="0.00043982" />
     </inertial>
     <visual>
@@ -86,5 +86,5 @@
     <limit
       lower="-2.618"
-      upper="2.618"
+      upper="2.168"
       effort="100"
       velocity="5" />
@@ -93,7 +93,7 @@
     name="link2">
     <inertial>
-      <origin xyz="0.21852 -0.00861 0.00126" rpy="0 0 0" />
-      <mass value="1.16" />
-      <inertia ixx="0.00111915" ixy="0.00182916" ixz="0.00019233" iyy="0.06763251" iyz="0.00000767" izz="0.067559" />
+      <origin xyz="0.198666145229743 -0.010926924140076 0.00142121714502687" rpy="0 0 0" />
+      <mass value="1.17" />
+      <inertia ixx="0.00116918" ixy="-0.00180037" ixz="0.00025146" iyy="0.06785384" iyz="-0.00000455" izz="0.06774489" />
     </inertial>
     <visual>
@@ -143,7 +143,7 @@
     name="link3">
     <inertial>
-      <origin xyz="-0.01999 -0.14808 -0.00053" rpy="0 0 0" />
+      <origin xyz="-0.0202737662122021 -0.133914995944595 -0.000458682652737356" rpy="0 0 0" />
       <mass value="0.5" />
-      <inertia ixx="0.01347608" ixy="0.00161034" ixz="0.00000066" iyy="0.00046377" iyz="0.00000162" izz="0.01363321" />
+      <inertia ixx="0.01361711" ixy="0.00165794" ixz="-0.00000048" iyy="0.00045024" iyz="-0.00000045" izz="0.01380322" />
     </inertial>
     <visual>
@@ -193,7 +193,7 @@
     name="link4">
     <inertial>
-      <origin xyz="0.00013 -0.00076 -0.00394" rpy="0 0 0" />
+      <origin xyz="-9.66635791618542E-05 0.000876064475651083 -0.00496880904640868" rpy="0 0 0" />
       <mass value="0.38" />
-      <inertia ixx="0.00017844" ixy="0.00000062" ixz="0.00000067" iyy="0.00018914" iyz="0.00000408" izz="0.00014613" />
+      <inertia ixx="0.00018501" ixy="0.00000054" ixz="0.00000120" iyy="0.00018965" iyz="-0.00000841" izz="0.00015484" />
     </inertial>
     <visual>
@@ -242,7 +242,7 @@
     name="link5">
     <inertial>
-      <origin xyz="0.00018 -0.06104 -0.00227" rpy="0 0 0" />
+      <origin xyz="-4.10554118924211E-05 -0.0566486692356075 -0.0037205791677906" rpy="0 0 0" />
       <mass value="0.383" />
-      <inertia ixx="0.00172318" ixy="0.00000259" ixz="0.00000010" iyy="0.00017936" iyz="0.00000990" izz="0.00171172" />
+      <inertia ixx="0.00166169" ixy="0.00000006" ixz="-0.00000007" iyy="0.00018510" iyz="0.00001026" izz="0.00164321" />
     </inertial>
     <visual>
@@ -291,7 +291,7 @@
     name="link6">
     <inertial>
-      <origin xyz="-0.00003 0.00006 0.04618" rpy="0 0 0" />
-      <mass value="0.007" />
-      <inertia ixx="0.00152112" ixy="0.00000202" ixz="0.00000261" iyy="0.00138626" iyz="0.00000002" izz="0.00031152" />
+      <origin xyz="-8.82590762930069E-05 9.0598378529832E-06 -0.002" rpy="0 0 0" />
+      <mass value="0.00699089613564366" />
+      <inertia ixx="5.73015540542155E-07" ixy="-1.98305403089247E-22" ixz="-7.2791893904596E-23" iyy="5.73015540542155E-07" iyz="-3.4146026640245E-24" izz="1.06738869138926E-06" />
     </inertial>
     <visual>

File: src/robot_description/piper_description/urdf/piper_no_gripper_description_gazebo.xacro (robot description, xacro)
@@ -44,7 +44,7 @@
     name="link1">
     <inertial>
-      <origin xyz="0.00032 -0.00041 -0.00348" rpy="0 0 0" />
-      <mass value="0.71" />
-      <inertia ixx="0.00050027" ixy="0.00000078" ixz="0.00000626" iyy="0.00040879" iyz="0.00000462" izz="0.00045802" />
+            <origin xyz="0.000121504734057468 0.000104632162460536 -0.00438597309559853" rpy="0 0 0" />
+            <mass value="0.71" />
+            <inertia ixx="0.00048916" ixy="-0.00000036" ixz="-0.00000224" iyy="0.00040472" iyz="-0.00000242" izz="0.00043982" />
     </inertial>
     <visual>
@@ -86,5 +86,5 @@
     <limit
       lower="-2.618"
-      upper="2.618"
+      upper="2.168"
       effort="100"
       velocity="5" />
@@ -93,7 +93,7 @@
     name="link2">
     <inertial>
-      <origin xyz="0.21852 -0.00861 0.00126" rpy="0 0 0" />
-      <mass value="1.16" />
-      <inertia ixx="0.00111915" ixy="0.00182916" ixz="0.00019233" iyy="0.06763251" iyz="0.00000767" izz="0.067559" />
+            <origin xyz="0.198666145229743 -0.010926924140076 0.00142121714502687" rpy="0 0 0" />
+            <mass value="1.17" />
+            <inertia ixx="0.00116918" ixy="-0.00180037" ixz="0.00025146" iyy="0.06785384" iyz="-0.00000455" izz="0.06774489" />
     </inertial>
     <visual>
@@ -143,7 +143,7 @@
     name="link3">
     <inertial>
-      <origin xyz="-0.01999 -0.14808 -0.00053" rpy="0 0 0" />
-      <mass value="0.5" />
-      <inertia ixx="0.01347608" ixy="0.00161034" ixz="0.00000066" iyy="0.00046377" iyz="0.00000162" izz="0.01363321" />
+            <origin xyz="-0.0202737662122021 -0.133914995944595 -0.000458682652737356" rpy="0 0 0" />
+            <mass value="0.5" />
+            <inertia ixx="0.01361711" ixy="0.00165794" ixz="-0.00000048" iyy="0.00045024" iyz="-0.00000045" izz="0.01380322" />
     </inertial>
     <visual>
@@ -193,7 +193,7 @@
     name="link4">
     <inertial>
-      <origin xyz="0.00013 -0.00076 -0.00394" rpy="0 0 0" />
-      <mass value="0.38" />
-      <inertia ixx="0.00017844" ixy="0.00000062" ixz="0.00000067" iyy="0.00018914" iyz="0.00000408" izz="0.00014613" />
+            <origin xyz="-9.66635791618542E-05 0.000876064475651083 -0.00496880904640868" rpy="0 0 0" />
+            <mass value="0.38" />
+            <inertia ixx="0.00018501" ixy="0.00000054" ixz="0.00000120" iyy="0.00018965" iyz="-0.00000841" izz="0.00015484" />
     </inertial>
     <visual>
@@ -242,7 +242,7 @@
     name="link5">
     <inertial>
-      <origin xyz="0.00018 -0.06104 -0.00227" rpy="0 0 0" />
-      <mass value="0.383" />
-      <inertia ixx="0.00172318" ixy="0.00000259" ixz="0.00000010" iyy="0.00017936" iyz="0.00000990" izz="0.00171172" />
+            <origin xyz="-4.10554118924211E-05 -0.0566486692356075 -0.0037205791677906" rpy="0 0 0" />
+            <mass value="0.383" />
+            <inertia ixx="0.00166169" ixy="0.00000006" ixz="-0.00000007" iyy="0.00018510" iyz="0.00001026" izz="0.00164321" />
     </inertial>
     <visual>
@@ -291,7 +291,7 @@
     name="link6">
     <inertial>
-      <origin xyz="-0.00003 0.00006 0.04618" rpy="0 0 0" />
-      <mass value="0.007" />
-      <inertia ixx="0.00152112" ixy="0.00000202" ixz="0.00000261" iyy="0.00138626" iyz="0.00000002" izz="0.00031152" />
+            <origin xyz="-8.82590762930069E-05 9.0598378529832E-06 -0.002" rpy="0 0 0" />
+            <mass value="0.00699089613564366" />
+            <inertia ixx="5.73015540542155E-07" ixy="-1.98305403089247E-22" ixz="-7.2791893904596E-23" iyy="5.73015540542155E-07" iyz="-3.4146026640245E-24" izz="1.06738869138926E-06" />
     </inertial>
     <visual>

File: src/robot_description/piper_description/urdf/piper_no_gripper_description_old.urdf (robot description, URDF)
Before this commit: robot piper, 7 links, 6 joints
Links:
- link link2: mass 1.16 -> 1.17
- link link6: mass 0.007 -> 0.00699089613564366
Joints:
- joint joint1: limit lower=-2.618 upper=2.618 effort=100 velocity=5 -> lower=-2.618 upper=2.168 effort=100 velocity=5
