Commit message: update piper x usd and add nero usd

File: src/robot_description/nero_description/urdf/nero_description.urdf (robot description, URDF)
Before this commit: robot nero_description, 8 links, 7 joints
Links:
- added link end_effector
- added link world
- link Link1: geometry collision mesh filename=package://nero_description/meshes/Link1.STL; visual mesh filename=package://nero_description/meshes/dae/link1.dae
- link Link2: geometry collision mesh filename=package://nero_description/meshes/Link2.STL; visual mesh filename=package://nero_description/meshes/dae/link2.dae
- link Link3: geometry collision mesh filename=package://nero_description/meshes/Link3.STL; visual mesh filename=package://nero_description/meshes/dae/link3.dae
- link Link4: geometry collision mesh filename=package://nero_description/meshes/Link4.STL; visual mesh filename=package://nero_description/meshes/dae/link4.dae
- link Link5: geometry collision mesh filename=package://nero_description/meshes/Link5.STL; visual mesh filename=package://nero_description/meshes/dae/link5.dae
- link Link6: geometry collision mesh filename=package://nero_description/meshes/Link6.STL; visual mesh filename=package://nero_description/meshes/dae/link6.dae
- link Link7: mass 0.00232665325657446 -> 0; geometry collision mesh filename=package://nero_description/meshes/Link7.STL; visual mesh filename=package://nero_description/meshes/dae/link7.dae
- link base_link: mass 0.487153985946125 -> 0.77; geometry collision mesh filename=package://nero_description/meshes/base_link.STL; visual mesh filename=package://nero_description/meshes/dae/base_link.dae
Joints:
- added joint end_effector_joint: type fixed, parent Link7, child end_effector, origin xyz=0.00000000 0.00000000 -0.02350000 rpy=0 0 0
- added joint world_to_base_link: type fixed, parent world, child base_link, origin xyz=0 0 0 rpy=0 0 0
- joint joint1: limit lower=-2.7402 upper=2.7402 effort=100 velocity=10 -> lower=-2.7 upper=2.7 effort=0 velocity=0
- joint joint2: axis 0 0 -1 -> 0 0 1; limit lower=-0.2618 upper=3.3161 effort=100 velocity=10 -> lower=-1.74 upper=1.74 effort=0 velocity=0; origin xyz=0 0 0 rpy=1.5708 1.5708 0 -> xyz=0 0 0 rpy=1.5708 3.1415 0
- joint joint3: limit lower=-2.7925 upper=2.7925 effort=100 velocity=10 -> lower=-2.75 upper=2.75 effort=0 velocity=0
- joint joint4: axis 0 0 -1 -> 0 0 1; limit lower=-1.0472 upper=2.1817 effort=100 velocity=10 -> lower=-1.01 upper=2.14 effort=0 velocity=0
- joint joint5: limit lower=-2.7925 upper=2.7925 effort=100 velocity=10 -> lower=-2.75 upper=2.75 effort=0 velocity=0
- joint joint6: axis 0 0 -1 -> 0 0 1; limit lower=-0.7505 upper=1.0123 effort=100 velocity=10 -> lower=-0.73 upper=0.95 effort=0 velocity=0
- joint joint7: limit lower=-1.57 upper=1.57 effort=100 velocity=10 -> lower=-1.57 upper=1.57 effort=0 velocity=0

File: src/robot_description/piper_x_description/urdf/piper_x_description_d435.urdf (robot description, URDF)
Before this commit: robot piper_x_camera, 13 links, 12 joints
Links:
- link camera_stand_link: geometry collision mesh filename=package://piper_x_description/meshes/dae/realsense_mid_stan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; visual mesh filename=package://piper_x_description/meshes/dae/realsense_mid_stan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

Commit message: 修改惯量矩阵

File: src/robot_description/nero_description/urdf/nero_description.urdf (robot description, URDF)
Before this commit: robot nero_description, 10 links, 9 joints
Links:
- link Link7: mass 0 -> 0.000001
