Commit message: 增加nero的末端支架

File: src/robot_description/nero_description/urdf/nero_description_stand_v2.urdf (robot description, URDF)
Before this commit: robot nero_description, 10 links, 9 joints
Links:
- link end_effector: geometry collision mesh filename=package://nero_description/meshes/stand_v2.dae; visual mesh filename=package://nero_description/meshes/stand_v2.dae
